File: power_supply.kicad_sch (KiCad schematic)
At the start: 38 parts, among them IC2 UCC3803DTR, Q1 MMBT42, Q2 FDS2672CT, SW1 SW_SPST

Commit message: Update inductor footprint
Parts:
- L2: footprint Inductor_SMD:L_CommonMode_Wurth_WE-CNSW-1206 -> eclectronics_nixie_footprints:WE-PD_1210
Changed lines of the file:
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@@
 			)
 		)
-		(property "Footprint" "Inductor_SMD:L_CommonMode_Wurth_WE-CNSW-1206"
+		(property "Footprint" "eclectronics_nixie_footprints:WE-PD_1210"
 			(at 153.67 76.2 0)
 			(effects
