File: nixie-tube-clock.kicad_pcb (KiCad board)
At the start: 2 copper layers, 157.5 x 72 mm, 143 parts, among them IC1 TPS61041DBVR, IC2 UCC3803DTR, J5 USB4105-GF-A, Q1 MMBT42, Q2 FDS2672CT, SW1 SW_SPST, U1 CD40109BPW, U2 W25Q32JV, U3 RP2350A, U4 MCP1702T-3302E_CB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

Commit message: Fix +160V clearance issues
Routing:
- net +5V: track 442.8 -> 458.3 mm
- net +3V3: track 153.1 -> 159.9 mm, vias 19 -> 20
- net Net-(N5-PadA): track 14.4 -> 12.8 mm

Commit message: Fix silkscreen overlap; add logo
Parts:
- added OlinLogoLg: G***, Eclectronics:OlinLogoLg, F.Cu at (264.0, 75.6)
- added svg2mod: G***, Eclectronics:OlinLogoHuge, F.Cu at (235.8, 67.9)
Changed lines of the file:
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@@
 		)
 	)
+	(footprint "Eclectronics:OlinLogoHuge"
+		(layer "F.Cu")
+		(at 235.824236 67.893135)
+		(descr "Imported from OlinLogoHuge.svg")
+		(tags "svg2mod")
+		(property "Reference" "svg2mod"
+			(at 0 -20.262994 0)
+			(layer "F.SilkS")
+			(hide yes)
+			(effects
+				(font
+					(size 1.524 1.524)
+					(thickness 0.3048)
+				)
+			)
+		)
+		(property "Value" "G***"
+			(at 0 20.262994 0)
+			(layer "F.SilkS")
+			(hide yes)
+			(effects
+				(font
+					(size 1.524 1.524)
+					(thickness 0.3048)
+				)
+			)
+		)
+		(property "Datasheet" ""
+			(at 0 0 0)
+			(layer "F.Fab")
+			(hide yes)
+			(effects
+				(font
+					(size 1.27 1.27)
+					(thickness 0.15)
+				)
+			)
+		)
+		(property "Description" ""
+			(at 0 0 0)
+			(layer "F.Fab")
+			(hide yes)
+			(effects
+				(font
+					(size 1.27 1.27)
+					(thickness 0.15)
+				)
+			)
+		)
+		(attr smd)
+		(fp_poly
+			(pts
+				(xy -13.863794 -15.351233) (xy -14.814854 -14.067888) (xy -15.292478 -12.358205) (xy -15.297825 -10.274876)
+				(xy -14.832055 -7.870594) (xy -13.896326 -5.198051) (xy -12.491797 -2.30994) (xy -10.619628 0.741047)
+				(xy -8.821038 3.214592) (xy -6.871892 5.555542) (xy -4.808179 7.73794) (xy -2.665891 9.73583) (xy -0.481017 11.523259)
+				(xy 1.710452 13.074268) (xy 3.872526 14.362904) (xy 5.969215 15.363211) (xy 7.964528 16.049232)
+				(xy 4.908466 16.197876) (xy 1.850561 16.209548) (xy -1.192083 16.0886) (xy -4.202363 15.839383)
+				(xy -7.163174 15.46625) (xy -10.057413 14.973551) (xy -12.867976 14.365639) (xy -15.577759 13.646864)
+				(xy -18.169659 12.82158) (xy -20.626572 11.894137) (xy -22.931394 10.868887) (xy -25.067021 9.750181)
+				(xy -27.016349 8.542372) (xy -28.762276 7.249811) (xy -30.287696 5.87685) (xy -31.575507 4.42784)
+				(xy -32.75661 2.637169) (xy -33.508679 0.850099) (xy -33.844885 -0.919738) (xy -33.778404 -2.658707)
+				(xy -33.322406 -4.353175) (xy -32.490067 -5.989508) (xy -31.294558 -7.554071) (xy -29.749052 -9.033231)
+				(xy -27.866724 -10.413354) (xy -25.660746 -11.680807) (xy -23.14429 -12.821955) (xy -20.330531 -13.823164)
+				(xy -17.232641 -14.670802) (xy -13.863794 -15.351233)
+			)
+			(stroke
+				(width 0)
+				(type solid)
+			)
+			(fill yes)
+			(layer "B.SilkS")
+		)
+		(fp_poly
+			(pts
+				(xy -7.964528 -16.04879) (xy -4.908549 -16.197512) (xy -1.850725 -16.209251) (xy 1.191841 -16.08836)
+				(xy 4.202045 -15.83919) (xy 7.162787 -15.466093) (xy 10.056963 -14.97342) (xy 12.86747 -14.365523)
+				(xy 15.577207 -13.646754) (xy 18.169071 -12.821464) (xy 20.62596 -11.894006) (xy 22.93077 -10.86873)
+				(xy 25.0664 -9.749988) (xy 27.015747 -8.542133) (xy 28.761708 -7.249514) (xy 30.287182 -5.876486)
+				(xy 31.575065 -4.427398) (xy 32.756244 -2.636728) (xy 33.508355 -0.849658) (xy 33.84458 0.920176)
+				(xy 33.778098 2.659139) (xy 33.322092 4.353597) (xy 32.489741 5.989914) (xy 31.294226 7.554457)
+				(xy 29.748729 9.03359) (xy 27.86643 10.413679) (xy 25.66051 11.681087) (xy 23.144149 12.822182)
+				(xy 20.33053 13.823328) (xy 17.232832 14.67089) (xy 13.864236 15.351233) (xy 14.815017 14.068051)
+				(xy 15.292533 12.358485) (xy 15.297896 10.275235) (xy 14.832218 7.871001) (xy 13.896613 5.198482)
+				(xy 12.492193 2.31038) (xy 10.62007 -0.740605) (xy 8.82145 -3.214281) (xy 6.872227 -5.555329) (xy 4.808409 -7.737792)
+				(xy 2.666003 -9.735716) (xy 0.48102 -11.523144) (xy -1.710534 -13.074121) (xy -3.872648 -14.362692)
+				(xy -5.969316 -15.3629) (xy -7.964528 -16.04879)
+			)
+			(stroke
+				(width 0)
+				(type solid)
+			)
+			(fill yes)
+			(layer "B.SilkS")
+		)
+		(embedded_fonts no)
+	)
 	(footprint "Resistor_SMD:R_2512_6332Metric"
 		(layer "F.Cu")
@@
 		)
 	)
+	(footprint "Eclectronics:OlinLogoLg"
+		(layer "F.Cu")
+		(at 264 75.6)
+		(descr "Imported from OlinLogo.svg")
+		(tags "svg2mod")
+		(property "Reference" "OlinLogoLg"
+			(at 0 -5.923376 0)
+			(layer "F.SilkS")
+			(hide yes)
+			(effects
+				(font
+					(size 1.524 1.524)
+					(thickness 0.3048)
+				)
+			)
+		)
+		(property "Value" "G***"
+			(at 0 5.923376 0)
+			(layer "F.SilkS")
+			(hide yes)
+			(effects
+				(font
+					(size 1.524 1.524)
+					(thickness 0.3048)
+				)
+			)
+		)
+		(property "Datasheet" ""
+			(at 0 0 0)
+			(layer "F.Fab")
+			(hide yes)
+			(effects
+				(font
+					(size 1.27 1.27)
+					(thickness 0.15)
+				)
+			)
+		)
+		(property "Description" ""
+			(at 0 0 0)
+			(layer "F.Fab")
+			(hide yes)
+			(effects
+				(font
+					(size 1.27 1.27)
+					(thickness 0.15)
+				)
+			)
+		)
+		(attr smd)
+		(fp_poly
+			(pts
+				(xy 1.330295 -2.680588) (xy 0.746852 -2.707093) (xy 0.163539 -2.703849) (xy -0.415379 -2.671942)
+				(xy -0.985637 -2.612457) (xy -1.542973 -2.526479) (xy -2.083123 -2.415092) (xy -2.601821 -2.279382)
+				(xy -3.094804 -2.120434) (xy -3.557808 -1.939332) (xy -3.986569 -1.737162) (xy -4.376823 -1.515008)
+				(xy -4.724306 -1.273956) (xy -5.024753 -1.015091) (xy -5.273902 -0.739497) (xy -5.497045 -0.390554)
+				(xy -5.623143 -0.042947) (xy -5.655691 0.299709) (xy -5.598185 0.633796) (xy -5.45412 0.955699)
+				(xy -5.226994 1.261801) (xy -4.920301 1.548486) (xy -4.537539 1.812138) (xy -4.082202 2.049139)
+				(xy -3.557787 2.255873) (xy -2.96779 2.428725) (xy -2.315708 2.564077) (xy -2.493292 2.306868) (xy -2.563324 1.95472)
+				(xy -2.526101 1.521611) (xy -2.381916 1.021519) (xy -2.131065 0.468423) (xy -1.773843 -0.123701)
+				(xy -1.43398 -0.587051) (xy -1.063231 -1.021678) (xy -0.670161 -1.421409) (xy -0.263333 -1.780072)
+				(xy 0.148691 -2.091494) (xy 0.557345 -2.349503) (xy 0.954068 -2.547925) (xy 1.330295 -2.680588)
+			)
+			(stroke
+				(width 0)
+				(type solid)
+			)
+			(fill yes)
+			(layer "F.SilkS")
+		)
+		(fp_poly
+			(pts
+				(xy 2.315634 -2.564077) (xy 2.493269 -2.306836) (xy 2.563316 -1.954668) (xy 2.526082 -1.521546)
+				(xy 2.381875 -1.021448) (xy 2.131001 -0.468349) (xy 1.773769 0.123775) (xy 1.433912 0.5871) (xy 1.063179 1.02171)
+				(xy 0.67013 1.421431) (xy 0.263323 1.78009) (xy -0.148682 2.091516) (xy -0.557326 2.349535) (xy -0.95405 2.547975)
+				(xy -1.330295 2.680662) (xy -0.746836 2.707152) (xy -0.163508 2.703896) (xy 0.415424 2.671979) (xy 0.985697 2.612486)
+				(xy 1.543046 2.526502) (xy 2.083206 2.415112) (xy 2.601913 2.279401) (xy 3.094903 2.120453) (xy 3.557911 1.939355)
+				(xy 3.986674 1.737191) (xy 4.376925 1.515045) (xy 4.724403 1.274003) (xy 5.024841 1.01515) (xy 5.273975 0.739571)
+				(xy 5.497105 0.390628) (xy 5.623196 0.04302) (xy 5.655742 -0.299636) (xy 5.598237 -0.633725) (xy 5.454174 -0.955631)
+				(xy 5.227049 -1.261737) (xy 4.920355 -1.548427) (xy 4.537585 -1.812086) (xy 4.082234 -2.049096)
+				(xy 3.557796 -2.255842) (xy 2.967765 -2.428708) (xy 2.315634 -2.564077)
+			)
+			(stroke
+				(width 0)
+				(type solid)
+			)
+			(fill yes)
+			(layer "F.SilkS")
+		)
+		(embedded_fonts no)
+	)
 	(footprint "Capacitor_SMD:C_0805_2012Metric_Pad1.18x1.45mm_HandSolder"
 		(layer "F.Cu")
@@
 		(tags "resistor")
 		(property "Reference" "R35"
-			(at 2.8326 0.6908 90)
+			(at 2.1922 0.5498 270)
 			(layer "F.SilkS")
 			(effects
@@
 		(net 2)
 		(net_name "GND")
+		(locked yes)
 		(layer "B.Cu")
 		(hatch edge 0.5)

Commit message: Misc final project updates
Other:
- outline, holes or cut-outs redrawn
- board text added: "Nixie Tube Clock V1.2 Eclectronics Mark Belanger & Carter Harris"
- board text removed: "Nixie Tube Clock V1.0 Eclectronics Mark Belanger & Carter Harris"
Changed lines of the file:
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@@
 		)
 	)
-	(gr_rect
-		(start 114.6356 41.6732)
-		(end 272.1356 113.6732)
+	(gr_line
+		(start 114.6356 109.8632)
+		(end 114.6356 45.4832)
 		(stroke
 			(width 0.05)
 			(type default)
 		)
-		(fill no)
+		(layer "Edge.Cuts")
+	)
+	(gr_arc
+		(start 114.6356 45.4832)
+		(mid 115.751523 42.789123)
+		(end 118.4456 41.6732)
+		(stroke
+			(width 0.05)
+			(type default)
+		)
+		(layer "Edge.Cuts")
+	)
+	(gr_line
+		(start 272.1356 45.4832)
+		(end 272.1356 109.8632)
+		(stroke
+			(width 0.05)
+			(type default)
+		)
+		(layer "Edge.Cuts")
+	)
+	(gr_arc
+		(start 118.4456 113.6732)
+		(mid 115.751523 112.557277)
+		(end 114.6356 109.8632)
+		(stroke
+			(width 0.05)
+			(type default)
+		)
+		(layer "Edge.Cuts")
+	)
+	(gr_line
+		(start 118.4456 41.6732)
+		(end 268.3256 41.6732)
+		(stroke
+			(width 0.05)
+			(type default)
+		)
+		(layer "Edge.Cuts")
+	)
+	(gr_arc
+		(start 272.1356 109.8632)
+		(mid 271.019677 112.557277)
+		(end 268.3256 113.6732)
+		(stroke
+			(width 0.05)
+			(type default)
+		)
+		(layer "Edge.Cuts")
+	)
+	(gr_arc
+		(start 268.3256 41.6732)
+		(mid 271.019677 42.789123)
+		(end 272.1356 45.4832)
+		(stroke
+			(width 0.05)
+			(type default)
+		)
+		(layer "Edge.Cuts")
+	)
+	(gr_line
+		(start 268.3256 113.6732)
+		(end 118.4456 113.6732)
+		(stroke
+			(width 0.05)
+			(type default)
+		)
 		(layer "Edge.Cuts")
 	)
@@
 		)
 	)
-	(gr_text "Nixie Tube Clock V1.0\nEclectronics\nMark Belanger & Carter Harris"
+	(gr_text "Nixie Tube Clock V1.2\nEclectronics\nMark Belanger & Carter Harris"
 		(at 270.3 84.9 0)
 		(layer "F.SilkS")
